File: SuperSpeakerSwitcher.sch (KiCad schematic (older format))
At the start: 58 parts, among them J1 Conn_01x03, J10 Conn_01x01, J11 Conn_01x01, J12 Conn_01x01, J13 Conn_01x01, J14 Conn_01x01, J15 Conn_01x01, J16 Conn_01x01, J17 Conn_01x01, J18 Conn_01x01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

Commit message: Alternate routing
Parts:
- added D5, D6: 1N4007, Diode_THT:D_DO-41_SOD81_P10.16mm_Horizontal, symbol Diode:1N4007
- added J23: Conn_01x03, Connectors_Terminal_Blocks:TerminalBlock_bornier-3_P5.08mm, symbol SuperSpeakerSwitcher-rescue:Conn_01x03
- C1: symbol CP -> SuperSpeakerSwitcher-rescue:CP
- C2, C3: symbol C_Small -> SuperSpeakerSwitcher-rescue:C_Small
- D1, D3: symbol LED -> SuperSpeakerSwitcher-rescue:LED
- D2, D4: symbol D -> SuperSpeakerSwitcher-rescue:D
- J1: symbol Conn_01x03 -> SuperSpeakerSwitcher-rescue:Conn_01x03
- J10, J11, J12, J13, J14, J15, J16, J17, J18, J19, J20, J21, J22, J3, J4, J5, J6, J7, J8, J9: symbol Conn_01x01 -> SuperSpeakerSwitcher-rescue:Conn_01x01
- J2: symbol Jack-DC -> SuperSpeakerSwitcher-rescue:Jack-DC
- Q1: symbol 2N3904 -> SuperSpeakerSwitcher-rescue:2N3904
- Q3: symbol TIP42 -> SuperSpeakerSwitcher-rescue:TIP42
- R1, R10, R11, R12, R2, R3, R4, R5, R7, R8, R9: symbol R -> SuperSpeakerSwitcher-rescue:R
- RLY1, RLY10, RLY11, RLY12, RLY13, RLY14, RLY15, RLY16, RLY2, RLY3, RLY4, RLY5, RLY6, RLY7, RLY8, RLY9: symbol SPDTRelay -> relay:SPDTRelay
Connections:
- wire segments 177 -> 182
