File: SuperSpeakerSwitcher.kicad_pcb (KiCad board)
At the start: 2 copper layers, 109 x 177 mm, 58 parts, among them J1 Conn_01x03, J10 Conn_01x01, J11 Conn_01x01, J12 Conn_01x01, J13 Conn_01x01, J14 Conn_01x01, J15 Conn_01x01, J16 Conn_01x01, J17 Conn_01x01, J18 Conn_01x01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

Commit message: Alternate routing
Parts:
- removed R10, R11, R12, R9: 8R, Resistors_THT:R_Axial_Power_L20.0mm_W6.4mm_P25.40mm
- added D5: 1N4007, Diode_THT:D_DO-41_SOD81_P10.16mm_Horizontal, F.Cu at (8.89, 221.0)
- added D6: 1N4007, Diode_THT:D_DO-41_SOD81_P10.16mm_Horizontal, F.Cu at (8.89, 206.6)
- Q3: value TIP42 -> TIP127
- moved J7 150.5 mm to (106.7, 154.9)
- moved J10 144.5 mm to (40.6, 154.9), turned to 180 degrees
- moved RLY9 124.2 mm to (109.2, 144.8)
- moved J17 120.8 mm to (35.6, 19.1), turned to 180 degrees
- moved J16 117.7 mm to (110.5, 19.1)
- moved J5 110.5 mm to (40.6, 81.3), turned to 180 degrees
- moved J11 109.2 mm to (86.4, 154.9)
- moved J4 107.8 mm to (106.7, 81.3)
- moved J14 103.2 mm to (61.0, 154.9), turned to 180 degrees
- moved RLY10 98.1 mm to (109.2, 130.8)
- moved J3 94.7 mm to (91.4, 92.7)
- moved RLY5 92.7 mm to (58.4, 71.1), turned to 180 degrees
- moved RLY6 91.7 mm to (58.4, 57.1), turned to 180 degrees
- moved J6 85.9 mm to (55.9, 92.7), turned to 180 degrees
- moved J15 83.3 mm to (110.5, 92.7)
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Connections:
- J1 pad 3: Net-(J1-Pad3) -> Net-(D5-Pad2)
- J2 pad 3: (no net) -> Net-(J2-Pad3)
- R1 pad 1: Net-(J1-Pad3) -> Net-(D5-Pad1)
Routing:
- net OUT2SPK2POS: track 415.8 -> 65.8 mm, vias 3 -> 0
- net OUT2SPK1POS: track 404.8 -> 64.8 mm, vias 3 -> 0
- net OUT1SPK1POS: track 347.6 -> 66.1 mm, vias 2 -> 0
- net OUT1SPK2POS: track 343.7 -> 64.9 mm, vias 2 -> 0
- net GND: track 415.8 -> 593.9 mm, vias 0 -> 2
- net COILV: track 369.7 -> 540.9 mm
- net OUT2SPK1NEG: track 188.6 -> 64.5 mm, vias 1 -> 0
- net OUT2SPK2NEG: track 179.0 -> 64.5 mm, vias 1 -> 0
- net OUT1SPK2NEG: track 173.5 -> 66.1 mm
- net OUT1SPK1NEG: track 169.4 -> 66.1 mm
- net AMP2SPK2NEG: track 129.1 -> 37.8 mm, vias 1 -> 0
- net AMP2SPK1NEG: track 126.0 -> 38.2 mm, vias 1 -> 0
- net AMP1SPK2NEG: track 117.6 -> 39.3 mm, vias 2 -> 0
- net AMP1SPK1NEG: track 113.8 -> 37.8 mm, vias 2 -> 0
- net AMP1SPK1POS: track 100.1 -> 37.8 mm
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Other:
- board text removed: "AMP1 SPK1 +"
- board text removed: "AMP1 SPK1 -"
- board text removed: "AMP1 SPK2 +"
- board text removed: "AMP1 SPK2 -"
- board text removed: "AMP2 SPK1 +"
- board text removed: "AMP2 SPK1 -"
- board text removed: "AMP2 SPK2 +"
- board text removed: "AMP2 SPK2 -"
- board text removed: "OUT1 SPK1 +"
- board text removed: "OUT1 SPK1 -"
- board text removed: "OUT1 SPK2 +"
- board text removed: "OUT1 SPK2 -"
- board text removed: "OUT2 SPK1 +"
- board text removed: "OUT2 SPK1 -"
- board text removed: "OUT2 SPK2 +"
- board text removed: "OUT2 SPK2 -"
- board text removed: "SUPER AUDIO SOURCE SWITCHER BY DANIEL MARKS CC-BY-SA 4.0"

Commit message: Remove erroneous diodes
Parts:
- removed D5, D6: 1N4007, Diode_THT:D_DO-41_SOD81_P10.16mm_Horizontal
Changed lines of the file:
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@@
     (tracks 275)
     (zones 0)
-    (modules 56)
-    (nets 31)
+    (modules 54)
+    (nets 30)
   )
   (page A4)
@@
   )
   (setup
-    (last_trace_width 1)
+    (last_trace_width 0.25)
     (user_trace_width 0.5)
     (user_trace_width 1)
@@
   (net 27 "Net-(D5-Pad2)")
   (net 28 "Net-(D5-Pad1)")
-  (net 29 "Net-(D6-Pad2)")
-  (net 30 "Net-(J2-Pad3)")
+  (net 29 "Net-(J2-Pad3)")
   (net_class Default "This is the default net class."
     (clearance 0.2)
@@
     (add_net "Net-(D5-Pad1)")
     (add_net "Net-(D5-Pad2)")
-    (add_net "Net-(D6-Pad2)")
     (add_net "Net-(J1-Pad3)")
     (add_net "Net-(J2-Pad3)")
@@
     (pad 1 thru_hole oval (at -2.54 0) (size 2.5 1.5) (drill oval 2 1.1) (layers *.Cu *.Mask)
       (net 7 AMP1SPK1POS))
-  )
-  (module Diode_THT:D_DO-41_SOD81_P10.16mm_Horizontal (layer F.Cu)
-    (at 8.89 206.57)
-    (descr "Diode, DO-41_SOD81 series, Axial, Horizontal, pin pitch=10.16mm, , length*diameter=5.2*2.7mm^2, , http://www.diodes.com/_files/packages/DO-41%20(Plastic).pdf")
-    (tags "Diode DO-41_SOD81 series Axial Horizontal pin pitch 10.16mm  length 5.2mm diameter 2.7mm")
-    (fp_text reference D6 (at 5.08 -2.47) (layer F.SilkS)
-      (effects (font (size 1 1) (thickness 0.15)))
-    )
-    (fp_text value 1N4007 (at 5.08 2.47) (layer F.Fab)
-      (effects (font (size 1 1) (thickness 0.15)))
-    )
-    (fp_text user K (at 0 -2.1) (layer F.SilkS)
-      (effects (font (size 1 1) (thickness 0.15)))
-    )
-    (fp_text user K (at 0 -2.1) (layer F.Fab)
-      (effects (font (size 1 1) (thickness 0.15)))
-    )
-    (fp_text user %R (at 59.69 0) (layer F.Fab)
-      (effects (font (size 1 1) (thickness 0.15)))
-    )
-    (fp_line (start 11.51 -1.6) (end -1.35 -1.6) (layer F.CrtYd) (width 0.05))
-    (fp_line (start 11.51 1.6) (end 11.51 -1.6) (layer F.CrtYd) (width 0.05))
-    (fp_line (start -1.35 1.6) (end 11.51 1.6) (layer F.CrtYd) (width 0.05))
-    (fp_line (start -1.35 -1.6) (end -1.35 1.6) (layer F.CrtYd) (width 0.05))
-    (fp_line (start 3.14 -1.47) (end 3.14 1.47) (layer F.SilkS) (width 0.12))
-    (fp_line (start 3.38 -1.47) (end 3.38 1.47) (layer F.SilkS) (width 0.12))
-    (fp_line (start 3.26 -1.47) (end 3.26 1.47) (layer F.SilkS) (width 0.12))
-    (fp_line (start 8.82 0) (end 7.8 0) (layer F.SilkS) (width 0.12))
-    (fp_line (start 1.34 0) (end 2.36 0) (layer F.SilkS) (width 0.12))
-    (fp_line (start 7.8 -1.47) (end 2.36 -1.47) (layer F.SilkS) (width 0.12))
-    (fp_line (start 7.8 1.47) (end 7.8 -1.47) (layer F.SilkS) (width 0.12))
-    (fp_line (start 2.36 1.47) (end 7.8 1.47) (layer F.SilkS) (width 0.12))
-    (fp_line (start 2.36 -1.47) (end 2.36 1.47) (layer F.SilkS) (width 0.12))
-    (fp_line (start 3.16 -1.35) (end 3.16 1.35) (layer F.Fab) (width 0.1))
-    (fp_line (start 3.36 -1.35) (end 3.36 1.35) (layer F.Fab) (width 0.1))
-    (fp_line (start 3.26 -1.35) (end 3.26 1.35) (layer F.Fab) (width 0.1))
-    (fp_line (start 10.16 0) (end 7.68 0) (layer F.Fab) (width 0.1))
-    (fp_line (start 0 0) (end 2.48 0) (layer F.Fab) (width 0.1))
-    (fp_line (start 7.68 -1.35) (end 2.48 -1.35) (layer F.Fab) (width 0.1))
-    (fp_line (start 7.68 1.35) (end 7.68 -1.35) (layer F.Fab) (width 0.1))
-    (fp_line (start 2.48 1.35) (end 7.68 1.35) (layer F.Fab) (width 0.1))
-    (fp_line (start 2.48 -1.35) (end 2.48 1.35) (layer F.Fab) (width 0.1))
-    (pad 2 thru_hole oval (at 10.16 0) (size 2.2 2.2) (drill 1.1) (layers *.Cu *.Mask)
-      (net 29 "Net-(D6-Pad2)"))
-    (pad 1 thru_hole rect (at 0 0) (size 2.2 2.2) (drill 1.1) (layers *.Cu *.Mask)
-      (net 28 "Net-(D5-Pad1)"))
-    (model ${KISYS3DMOD}/Diode_THT.3dshapes/D_DO-41_SOD81_P10.16mm_Horizontal.wrl
-      (at (xyz 0 0 0))
-      (scale (xyz 1 1 1))
-      (rotate (xyz 0 0 0))
-    )
-  )
-  (module Diode_THT:D_DO-41_SOD81_P10.16mm_Horizontal (layer F.Cu)
-    (at 8.89 220.98)
-    (descr "Diode, DO-41_SOD81 series, Axial, Horizontal, pin pitch=10.16mm, , length*diameter=5.2*2.7mm^2, , http://www.diodes.com/_files/packages/DO-41%20(Plastic).pdf")
-    (tags "Diode DO-41_SOD81 series Axial Horizontal pin pitch 10.16mm  length 5.2mm diameter 2.7mm")
-    (fp_text reference D5 (at 5.08 -2.47) (layer F.SilkS)
-      (effects (font (size 1 1) (thickness 0.15)))
-    )
-    (fp_text value 1N4007 (at 5.08 2.47) (layer F.Fab)
-      (effects (font (size 1 1) (thickness 0.15)))
-    )
-    (fp_text user K (at 0 -2.1) (layer F.SilkS)
-      (effects (font (size 1 1) (thickness 0.15)))
-    )
-    (fp_text user K (at 0 -2.1) (layer F.Fab)
-      (effects (font (size 1 1) (thickness 0.15)))
-    )
-    (fp_text user %R (at 5.47 0) (layer F.Fab)
-      (effects (font (size 1 1) (thickness 0.15)))
-    )
-    (fp_line (start 11.51 -1.6) (end -1.35 -1.6) (layer F.CrtYd) (width 0.05))
-    (fp_line (start 11.51 1.6) (end 11.51 -1.6) (layer F.CrtYd) (width 0.05))
-    (fp_line (start -1.35 1.6) (end 11.51 1.6) (layer F.CrtYd) (width 0.05))
-    (fp_line (start -1.35 -1.6) (end -1.35 1.6) (layer F.CrtYd) (width 0.05))
-    (fp_line (start 3.14 -1.47) (end 3.14 1.47) (layer F.SilkS) (width 0.12))
-    (fp_line (start 3.38 -1.47) (end 3.38 1.47) (layer F.SilkS) (width 0.12))
-    (fp_line (start 3.26 -1.47) (end 3.26 1.47) (layer F.SilkS) (width 0.12))
-    (fp_line (start 8.82 0) (end 7.8 0) (layer F.SilkS) (width 0.12))
-    (fp_line (start 1.34 0) (end 2.36 0) (layer F.SilkS) (width 0.12))
-    (fp_line (start 7.8 -1.47) (end 2.36 -1.47) (layer F.SilkS) (width 0.12))
-    (fp_line (start 7.8 1.47) (end 7.8 -1.47) (layer F.SilkS) (width 0.12))
-    (fp_line (start 2.36 1.47) (end 7.8 1.47) (layer F.SilkS) (width 0.12))
-    (fp_line (start 2.36 -1.47) (end 2.36 1.47) (layer F.SilkS) (width 0.12))
-    (fp_line (start 3.16 -1.35) (end 3.16 1.35) (layer F.Fab) (width 0.1))
-    (fp_line (start 3.36 -1.35) (end 3.36 1.35) (layer F.Fab) (width 0.1))
-    (fp_line (start 3.26 -1.35) (end 3.26 1.35) (layer F.Fab) (width 0.1))
-    (fp_line (start 10.16 0) (end 7.68 0) (layer F.Fab) (width 0.1))
-    (fp_line (start 0 0) (end 2.48 0) (layer F.Fab) (width 0.1))
-    (fp_line (start 7.68 -1.35) (end 2.48 -1.35) (layer F.Fab) (width 0.1))
-    (fp_line (start 7.68 1.35) (end 7.68 -1.35) (layer F.Fab) (width 0.1))
-    (fp_line (start 2.48 1.35) (end 7.68 1.35) (layer F.Fab) (width 0.1))
-    (fp_line (start 2.48 -1.35) (end 2.48 1.35) (layer F.Fab) (width 0.1))
-    (pad 2 thru_hole oval (at 10.16 0) (size 2.2 2.2) (drill 1.1) (layers *.Cu *.Mask)
-      (net 27 "Net-(D5-Pad2)"))
-    (pad 1 thru_hole rect (at 0 0) (size 2.2 2.2) (drill 1.1) (layers *.Cu *.Mask)
-      (net 28 "Net-(D5-Pad1)"))
-    (model ${KISYS3DMOD}/Diode_THT.3dshapes/D_DO-41_SOD81_P10.16mm_Horizontal.wrl
-      (at (xyz 0 0 0))
-      (scale (xyz 1 1 1))
-      (rotate (xyz 0 0 0))
-    )
   )
   (module Connectors:1pin (layer F.Cu)
@@
       (net 2 GND))
     (pad 3 thru_hole rect (at -3 4.7 90) (size 3.5 3.5) (drill oval 3 1) (layers *.Cu *.Mask)
-      (net 30 "Net-(J2-Pad3)"))
+      (net 29 "Net-(J2-Pad3)"))
   )
   (module TO_SOT_Packages_THT:TO-92_Inline_Wide (layer F.Cu)
@@
     (effects (font (size 1.5 1.5) (thickness 0.3)))
   )
-  (via (at 72.39 149.86) (size 0.6) (drill 0.4) (layers F.Cu B.Cu) (net 2))
   (segment (start 48.5 173) (end 50.5 173) (width 1) (layer B.Cu) (net 1))
   (segment (start 53 175.5) (end 53 182.5) (width 1) (layer B.Cu) (net 1))
@@
   (segment (start 70 167) (end 73.5 167) (width 1) (layer B.Cu) (net 1))
   (segment (start 98.83 180.25) (end 99 180.08) (width 1) (layer F.Cu) (net 1) (status 30))
+  (via (at 72.39 149.86) (size 0.6) (drill 0.4) (layers F.Cu B.Cu) (net 2))
   (segment (start 87.4 183.91) (end 87.25 183.91) (width 1) (layer F.Cu) (net 2))
   (segment (start 87.25 183.91) (end 84.74 186.42) (width 1) (layer F.Cu) (net 2))
